File: v0.3.brd (EAGLE design)
At the start: 50 x 50 mm, 36 parts, among them IC1 ESP-WROOM-02FRONT-FACE, Q2 BSA223SP, T1 BC846, T2 BC846

Commit message: slight cosmetic update and added gitignore
Parts:
- G1: value AB9V -> LI3V7; device battery:AB9V -> battery:LI3V7
Routing:
- net PROG: track 12.1 -> 12.8 mm
Changed lines of the file:
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@@
 <attribute name="VALUE" x="26.45" y="17.28" size="1.016" layer="27"/>
 </element>
-<element name="G1" library="battery" package="AB9V" value="AB9V" x="5.556" y="25.226" smashed="yes" rot="R180">
-<attribute name="NAME" x="9.366" y="27.766" size="1.27" layer="25" ratio="10" rot="R270"/>
+<element name="G1" library="battery" package="LI3V7" value="LI3V7" x="5.556" y="25.226" smashed="yes" rot="R180">
 <attribute name="VALUE" x="1.111" y="27.766" size="1.27" layer="27" ratio="10" rot="R270"/>
 </element>
@@
 <contactref element="U$2" pad="9"/>
 <wire x1="20.75" y1="17.12" x2="20.852" y2="17.018" width="0.254" layer="1"/>
-<wire x1="20.852" y1="17.018" x2="24.638" y2="17.272" width="0.254" layer="1"/>
-<via x="24.638" y="17.272" extent="1-16" drill="0.5"/>
-<wire x1="24.638" y1="17.272" x2="24.638" y2="10.668" width="0.254" layer="16"/>
-<via x="24.638" y="10.668" extent="1-16" drill="0.5"/>
-<wire x1="24.638" y1="10.668" x2="24.691" y2="10.975" width="0.254" layer="1"/>
-<wire x1="24.691" y1="10.975" x2="25.9299" y2="10.975" width="0.254" layer="1"/>
+<wire x1="20.852" y1="17.018" x2="20.828" y2="17.018" width="0.254" layer="1"/>
+<wire x1="20.828" y1="17.018" x2="20.828" y2="17.526" width="0.254" layer="1"/>
+<wire x1="20.828" y1="17.526" x2="24.13" y2="17.526" width="0.254" layer="1"/>
+<via x="24.13" y="17.526" extent="1-16" drill="0.5"/>
+<wire x1="24.13" y1="17.526" x2="24.13" y2="10.668" width="0.254" layer="16"/>
+<via x="24.13" y="10.668" extent="1-16" drill="0.5"/>
+<wire x1="24.13" y1="10.668" x2="24.437" y2="10.975" width="0.254" layer="1"/>
+<wire x1="24.437" y1="10.975" x2="25.9299" y2="10.975" width="0.254" layer="1"/>
 </signal>
 <signal name="N$10">
